File: semiactive/semiactive.kicad_pcb (KiCad board)
At the start: 2 copper layers, 85 x 85 mm, 12 parts, among them J1 5223004-2, U1 Teensy4.1

Commit message: DAQ updates
Other:
- board text added: "{dblquote}Oh, I want to be a stripper!{dblquote} - @Lauren Jones"
- board text removed: "{dblquote}Laurenitis{dblquote} - @Lauren Jones"
Changed lines of the file:
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@@
     (effects (font (size 1 1) (thickness 0.15)) (justify left bottom mirror))
   )
-  (gr_text "{dblquote}MILF slayer energy{dblquote}\n- @lucia" (at 139.446 76.962) (layer "B.SilkS")
+  (gr_text "{dblquote}MILF slayer energy{dblquote}\n- @lucia" (at 140.208 76.962) (layer "B.SilkS")
     (effects (font (size 1 1) (thickness 0.15)) (justify left bottom mirror))
   )
-  (gr_text "{dblquote}Laurenitis{dblquote} \n- @Lauren Jones" (at 132.588 71.628) (layer "B.SilkS")
+  (gr_text "{dblquote}Oh, I want to be a stripper!{dblquote} \n- @Lauren Jones" (at 138.176 71.882) (layer "B.SilkS")
     (effects (font (size 1 1) (thickness 0.15)) (justify left bottom mirror))
   )
