File: daq-wireless/daq-wireless.kicad_sch (KiCad schematic)
At the start: 34 parts, among them J1 5223004-2, J2 Micro_SD_Card, J3 USB_C_Receptacle_USB2.0, Q1 MMBT3904, Q2 MMBT3904, SW1 RESET, U1 ESP32-WROOM-32, U2 AMS1117, U3 FT231XS, U5 Ebyte_E01-ML01SP4

Commit message: Update SD symbol
Parts:
- removed J2: Micro_SD_Card, Connector_Card:microSD_HC_Hirose_DM3AT-SF-PEJM5, symbol Connector:Micro_SD_Card
- added J2: Micro_SD_Card, Connector_Card:microSD_HC_Hirose_DM3AT-SF-PEJM5, symbol Connector:Micro_SD_Card_Det_Hirose_DM3AT
- C10: value .1uF -> 1uF
Connections:
- net +3V3: now also J2.4 (VDD)
- net GND: now also J2.11 (SHIELD), J2.6 (VSS)
- net SD0: now also J2.7 (DAT0)
- net SD1: now also J2.8 (DAT1)
- net SD2: now also J2.1 (DAT2)
- net SD3: now also J2.2 (DAT3/CD)
- net SD_CLK: now also J2.5 (CLK)
- net SD_CMD: now also J2.3 (CMD)
- no-connect marks 33 -> 35
Changed lines of the file:
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@@
   (no_connect (at 118.11 77.47))
   (no_connect (at 37.465 67.31))
+  (no_connect (at 227.965 28.575))
   (no_connect (at 148.59 92.71))
   (no_connect (at 37.465 59.69))
@@
   (no_connect (at 118.11 85.09))
   (no_connect (at 123.19 178.435))
+  (no_connect (at 227.965 31.115))
   (no_connect (at 37.465 72.39))
   (no_connect (at 118.11 82.55))
@@
     )
   )
+  (symbol (lib_id "Connector:Micro_SD_Card_Det_Hirose_DM3AT") (at 205.105 41.275 180) (unit 1)
+    (in_bom yes) (on_board yes) (dnp no) (fields_autoplaced)
+    (property "Reference" "J2" (at 204.47 19.05 0)
+      (effects (font (size 1.27 1.27)))
+    )
+    (property "Value" "Micro_SD_Card" (at 204.47 21.59 0)
+      (effects (font (size 1.27 1.27)))
+    )
+    (property "Footprint" "Connector_Card:microSD_HC_Hirose_DM3AT-SF-PEJM5" (at 153.035 59.055 0)
+      (effects (font (size 1.27 1.27)) hide)
+    )
+    (property "Datasheet" "https://www.hirose.com/product/en/download_file/key_name/DM3/category/Catalog/doc_file_id/49662/?file_category_id=4&item_id=195&is_series=1" (at 205.105 43.815 0)
+      (effects (font (size 1.27 1.27)) hide)
+    )
+    (property "DPN" "HR1964CT-ND" (at 205.105 41.275 0)
+      (effects (font (size 1.27 1.27)) hide)
+    )
+    (pin "1")
+    (pin "10")
+    (pin "11")
+    (pin "2")
+    (pin "3")
+    (pin "4")
+    (pin "5")
+    (pin "6")
+    (pin "7")
+    (pin "8")
+    (pin "9")
+    (instances
+      (project "daq-wireless"
+        (path "/d87b4a87-5883-4edc-9ed5-8b7902b6705b"
+          (reference "J2") (unit 1)
+        )
+      )
+    )
+  )
   (symbol (lib_id "Device:C") (at 106.68 50.8 0) (unit 1)
     (in_bom yes) (on_board yes) (dnp no) (fields_autoplaced)
@@
       (effects (font (size 1.27 1.27)) (justify left))
     )
-    (property "Value" ".1uF" (at 110.49 52.705 0)
+    (property "Value" "1uF" (at 110.49 52.705 0)
       (effects (font (size 1.27 1.27)) (justify left))
     )
@@
         )
       )
-    )
-  )
-  (symbol (lib_id "Connector:Micro_SD_Card") (at 205.105 43.815 180) (unit 1)
-    (in_bom yes) (on_board yes) (dnp no) (fields_autoplaced)
-    (property "Reference" "J2" (at 204.47 21.59 0)
-      (effects (font (size 1.27 1.27)))
-    )
-    (property "Value" "Micro_SD_Card" (at 204.47 24.13 0)
-      (effects (font (size 1.27 1.27)))
-    )
-    (property "Footprint" "Connector_Card:microSD_HC_Hirose_DM3AT-SF-PEJM5" (at 175.895 51.435 0)
-      (effects (font (size 1.27 1.27)) hide)
-    )
-    (property "Datasheet" "http://katalog.we-online.de/em/datasheet/693072010801.pdf" (at 205.105 43.815 0)
-      (effects (font (size 1.27 1.27)) hide)
-    )
-    (property "DPN" "HR1964CT-ND" (at 205.105 43.815 0)
-      (effects (font (size 1.27 1.27)) hide)
-    )
-    (pin "1")
-    (pin "2")
-    (pin "3")
-    (pin "4")
-    (pin "5")
-    (pin "6")
-    (pin "7")
-    (pin "8")
-    (pin "9")
-    (instances
-      (project "daq-wireless"
-        (path "/d87b4a87-5883-4edc-9ed5-8b7902b6705b"
-          (reference "J2") (unit 1)
-        )
-      )

Commit message: Change CE pin away from UART tx
Connections:
- net ARGB: now also U1.11 (IO26); no longer U1.10 (IO25)
- net RADIO_CE: now also U1.10 (IO25); no longer U1.28 (IO17)
Changed lines of the file:
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@@
   (no_connect (at 148.59 105.41))
   (no_connect (at 118.11 77.47))
+  (no_connect (at 148.59 74.93))
   (no_connect (at 37.465 67.31))
   (no_connect (at 227.965 28.575))
-  (no_connect (at 148.59 92.71))
   (no_connect (at 37.465 59.69))
   (no_connect (at 123.19 163.195))
@@
     (stroke (width 0) (type default))
   )
+  (wire (pts (xy 148.59 92.71) (xy 151.13 92.71))
+    (stroke (width 0) (type default))
+  )
   (wire (pts (xy 59.69 153.67) (xy 59.69 155.575))
     (stroke (width 0) (type default))
@@
   )
   (wire (pts (xy 210.185 91.44) (xy 215.265 91.44))
-    (stroke (width 0) (type default))
-  )
-  (wire (pts (xy 151.13 74.93) (xy 148.59 74.93))
     (stroke (width 0) (type default))
   )
@@
     (effects (font (size 1.27 1.27)) (justify right bottom))
   )
+  (label "ARGB" (at 151.13 92.71 0) (fields_autoplaced)
+    (effects (font (size 1.27 1.27)) (justify left bottom))
+  )
   (label "D-" (at 51.435 161.29 0) (fields_autoplaced)
     (effects (font (size 1.27 1.27)) (justify left bottom))
@@
     (effects (font (size 1.27 1.27)) (justify left bottom))
   )
-  (label "RADIO_CE" (at 151.13 74.93 0) (fields_autoplaced)
-    (effects (font (size 1.27 1.27)) (justify left bottom))
-  )
   (label "RXD" (at 151.13 49.53 0) (fields_autoplaced)
     (effects (font (size 1.27 1.27)) (justify left bottom))
@@
     (effects (font (size 1.27 1.27)) (justify left bottom))
   )
-  (label "ARGB" (at 151.13 90.17 0) (fields_autoplaced)
-    (effects (font (size 1.27 1.27)) (justify left bottom))
-  )
   (label "EN" (at 262.89 80.645 0) (fields_autoplaced)
     (effects (font (size 1.27 1.27)) (justify left bottom))
@@
     (effects (font (size 1.27 1.27)) (justify left bottom))
   )
+  (label "RADIO_CE" (at 151.13 90.17 0) (fields_autoplaced)
+    (effects (font (size 1.27 1.27)) (justify left bottom))
+  )

Commit message: BOM
Parts:
- C1, C10, C3, C7, C9: DPN (none) -> 1276-1043-1-ND
- C10: footprint Capacitor_SMD:C_0402_1005Metric -> Capacitor_SMD:C_0603_1608Metric; DPN (none) -> 1276-1102-1-ND
- C2, C6, C8: DPN (none) -> 1276-1102-1-ND
- C4, C5: DPN (none) -> 1276-6460-1-ND
- C8: DPN (none) -> 1276-1119-1-ND
- R1, R4, R7, R8, R9: DPN (none) -> 1292-WR06X103JTLCT-ND
- R2, R3: DPN (none) -> RMCF0603JT5K10CT-ND
- R5, R6: DPN (none) -> 1292-WR06X102JTLCT-ND
- SW1: DPN (none) -> 2223-TS02-66-43-BK-160-LCR-D-ND
Changed lines of the file:
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@@
+      (effects (font (size 1.27 1.27)) hide)
+    )
+    (property "DPN" "1276-6460-1-ND" (at 244.475 142.24 0)
       (effects (font (size 1.27 1.27)) hide)
     )
@@
       (effects (font (size 1.27 1.27)) hide)
     )
+    (property "DPN" "1276-1102-1-ND" (at 83.185 136.525 0)
+      (effects (font (size 1.27 1.27)) hide)
+    )
     (pin "1")
     (pin "2")
@@
     )
     (property "Datasheet" "~" (at 257.81 74.93 0)
+      (effects (font (size 1.27 1.27)) hide)
+    )
+    (property "DPN" "1292-WR06X103JTLCT-ND" (at 257.81 74.93 0)
       (effects (font (size 1.27 1.27)) hide)
     )
@@
       (effects (font (size 1.27 1.27)) (justify left))
     )
-    (property "Footprint" "Capacitor_SMD:C_0402_1005Metric" (at 107.6452 54.61 0)
+    (property "Footprint" "Capacitor_SMD:C_0603_1608Metric" (at 107.6452 54.61 0)
       (effects (font (size 1.27 1.27)) hide)
     )
     (property "Datasheet" "~" (at 106.68 50.8 0)
+      (effects (font (size 1.27 1.27)) hide)
+    )
+    (property "DPN" "1276-1102-1-ND" (at 106.68 50.8 0)
       (effects (font (size 1.27 1.27)) hide)
     )
@@
       (effects (font (size 1.27 1.27)) hide)
     )
-    (property "DPN" "" (at 252.73 103.505 0)
+    (property "DPN" "1292-WR06X103JTLCT-ND" (at 252.73 103.505 0)
       (effects (font (size 1.27 1.27)) hide)
     )
@@
       (effects (font (size 1.27 1.27)) hide)
     )
+    (property "DPN" "1276-1119-1-ND" (at 227.33 81.915 0)
+      (effects (font (size 1.27 1.27)) hide)
+    )
     (pin "1")
     (pin "2")
@@
       (effects (font (size 1.27 1.27)) hide)
     )
-    (property "DPN" "" (at 140.335 159.385 0)
+    (property "DPN" "1292-WR06X102JTLCT-ND" (at 140.335 159.385 0)
       (effects (font (size 1.27 1.27)))
     )
@@
       (effects (font (size 1.27 1.27)) hide)
     )
+    (property "DPN" "1276-6460-1-ND" (at 219.075 142.24 0)
+      (effects (font (size 1.27 1.27)) hide)
+    )
     (pin "1")
     (pin "2")
@@
     )
     (property "Datasheet" "~" (at 85.09 182.245 0)
+      (effects (font (size 1.27 1.27)) hide)
+    )
+    (property "DPN" "1276-1043-1-ND" (at 85.09 182.245 0)
       (effects (font (size 1.27 1.27)) hide)
     )
@@
       (effects (font (size 1.27 1.27)) hide)
     )
+    (property "DPN" "RMCF0603JT5K10CT-ND" (at 55.88 151.13 0)
+      (effects (font (size 1.27 1.27)) hide)
+    )
     (pin "1")
     (pin "2")
@@
     )
     (property "Datasheet" "~" (at 240.665 42.545 0)
+      (effects (font (size 1.27 1.27)) hide)
+    )
+    (property "DPN" "1276-1043-1-ND" (at 240.665 42.545 0)
       (effects (font (size 1.27 1.27)) hide)
     )
@@
       (effects (font (size 1.27 1.27)) hide)
     )
+    (property "DPN" "1276-1043-1-ND" (at 215.265 81.915 0)
+      (effects (font (size 1.27 1.27)) hide)
+    )
     (pin "1")
     (pin "2")
@@
       (effects (font (size 1.27 1.27)) hide)
     )
+    (property "DPN" "1292-WR06X103JTLCT-ND" (at 180.975 135.255 0)
+      (effects (font (size 1.27 1.27)) hide)
+    )
     (pin "1")
     (pin "2")
@@
     )
     (property "Datasheet" "~" (at 125.095 36.195 0)
+      (effects (font (size 1.27 1.27)) hide)
+    )
+    (property "DPN" "1276-1043-1-ND" (at 125.095 36.195 0)
       (effects (font (size 1.27 1.27)) hide)
     )
@@
     )
     (property "Datasheet" "~" (at 113.665 36.195 0)
+      (effects (font (size 1.27 1.27)) hide)
+    )
+    (property "DPN" "1276-1102-1-ND" (at 113.665 36.195 0)
       (effects (font (size 1.27 1.27)) hide)
     )
@@
       (effects (font (size 1.27 1.27)) hide)
     )
+    (property "DPN" "2223-TS02-66-43-BK-160-LCR-D-ND" (at 250.19 80.645 0)
+      (effects (font (size 1.27 1.27)) hide)
+    )
     (pin "1")
     (pin "2")
@@
       (effects (font (size 1.27 1.27)) hide)
     )
-    (property "DPN" "" (at 252.73 111.125 0)
+    (property "DPN" "1292-WR06X103JTLCT-ND" (at 252.73 111.125 0)
       (effects (font (size 1.27 1.27)) hide)
     )
@@
     )
     (property "Datasheet" "~" (at 180.975 151.765 0)
+      (effects (font (size 1.27 1.27)) hide)
+    )
+    (property "DPN" "1292-WR06X103JTLCT-ND" (at 180.975 151.765 0)
       (effects (font (size 1.27 1.27)) hide)
     )
@@
       (effects (font (size 1.27 1.27)) hide)
     )
-    (property "DPN" "" (at 150.495 159.385 0)
+    (property "DPN" "1292-WR06X102JTLCT-ND" (at 150.495 159.385 0)
       (effects (font (size 1.27 1.27)))
     )
@@
     )
     (property "Datasheet" "~" (at 94.615 136.525 0)
+      (effects (font (size 1.27 1.27)) hide)
+    )
+    (property "DPN" "1276-1043-1-ND" (at 94.615 136.525 0)
       (effects (font (size 1.27 1.27)) hide)
     )
@@
     )
     (property "Datasheet" "~" (at 252.73 42.545 0)
+      (effects (font (size 1.27 1.27)) hide)
+    )
+    (property "DPN" "1276-1102-1-ND" (at 252.73 42.545 0)
       (effects (font (size 1.27 1.27)) hide)
     )
@@
       (effects (font (size 1.27 1.27)) hide)
     )
+    (property "DPN" "RMCF0603JT5K10CT-ND" (at 55.88 153.67 0)
+      (effects (font (size 1.27 1.27)) hide)
+    )

Commit message: Bugfix DAQ board
Parts:
- removed R9: 10k, Resistor_SMD:R_0603_1608Metric, symbol Device:R
- R8: now fitted; now in the parts list
Connections:
- net SD0 is gone; now on net IO0: J2.7 (DAT0), R8.2, U1.24 (IO2)
Changed lines of the file:
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@@
   (junction (at 125.095 32.385) (diameter 0) (color 0 0 0 0)
   )
-  (junction (at 252.73 107.315) (diameter 0) (color 0 0 0 0)
-  )
   (junction (at 257.81 80.645) (diameter 0) (color 0 0 0 0)
   )
@@
   (junction (at 83.185 140.335) (diameter 0) (color 0 0 0 0)
   )
+  (junction (at 158.115 52.07) (diameter 0) (color 0 0 0 0)
+  )
   (junction (at 227.33 91.44) (diameter 0) (color 0 0 0 0)
   )
@@
   )
   (junction (at 48.895 166.37) (diameter 0) (color 0 0 0 0)
+  )
+  (junction (at 158.115 46.99) (diameter 0) (color 0 0 0 0)
   )
   (junction (at 173.99 151.765) (diameter 0) (color 0 0 0 0)
@@
     (stroke (width 0) (type default))
   )
-  (wire (pts (xy 151.13 46.99) (xy 148.59 46.99))
+  (wire (pts (xy 161.29 46.99) (xy 158.115 46.99))
     (stroke (width 0) (type default))
   )
@@
   )
   (wire (pts (xy 151.13 85.09) (xy 148.59 85.09))
+    (stroke (width 0) (type default))
+  )
+  (wire (pts (xy 158.115 52.07) (xy 148.59 52.07))
     (stroke (width 0) (type default))
   )
@@
     (stroke (width 0.254) (type default))
   )
-  (wire (pts (xy 151.13 52.07) (xy 148.59 52.07))
+  (wire (pts (xy 161.29 52.07) (xy 158.115 52.07))
     (stroke (width 0) (type default))
   )
@@
     (stroke (width 0) (type default))
   )
+  (wire (pts (xy 158.115 46.99) (xy 158.115 52.07))
+    (stroke (width 0) (type default))
+  )
+  (wire (pts (xy 158.115 46.99) (xy 148.59 46.99))
+    (stroke (width 0) (type default))
+  )
   (wire (pts (xy 65.405 100.33) (xy 71.755 100.33))
     (stroke (width 0.254) (type default))
@@
     (effects (font (size 1.27 1.27)) (justify right bottom))
   )
-  (label "SD0" (at 151.13 52.07 0) (fields_autoplaced)
+  (label "SD0" (at 161.29 52.07 0) (fields_autoplaced)
     (effects (font (size 1.27 1.27)) (justify left bottom))
   )
@@
     (effects (font (size 1.27 1.27)) (justify left bottom))
   )
-  (label "IO0" (at 151.13 46.99 0) (fields_autoplaced)
+  (label "IO0" (at 161.29 46.99 0) (fields_autoplaced)
     (effects (font (size 1.27 1.27)) (justify left bottom))
   )
@@
     )
   )
-  (symbol (lib_id "power:GND") (at 252.73 114.935 0) (unit 1)
-    (in_bom yes) (on_board yes) (dnp no) (fields_autoplaced)
-    (property "Reference" "#PWR029" (at 252.73 121.285 0)
-      (effects (font (size 1.27 1.27)) hide)
-    )
-    (property "Value" "GND" (at 252.73 120.015 0)
-      (effects (font (size 1.27 1.27)))
-    )
-    (property "Footprint" "" (at 252.73 114.935 0)
-      (effects (font (size 1.27 1.27)) hide)
-    )
-    (property "Datasheet" "" (at 252.73 114.935 0)
-      (effects (font (size 1.27 1.27)) hide)
-    )
-    (pin "1")
-    (instances
-      (project "daq-wireless"
-        (path "/d87b4a87-5883-4edc-9ed5-8b7902b6705b"
-          (reference "#PWR029") (unit 1)
-        )
-      )
-    )
-  )
   (symbol (lib_id "Device:R") (at 257.81 74.93 0) (unit 1)
     (in_bom yes) (on_board yes) (dnp no) (fields_autoplaced)
@@
   )
   (symbol (lib_id "Device:R") (at 252.73 103.505 0) (unit 1)
-    (in_bom no) (on_board yes) (dnp yes) (fields_autoplaced)
+    (in_bom yes) (on_board yes) (dnp no) (fields_autoplaced)
     (property "Reference" "R8" (at 255.27 102.87 0)
       (effects (font (size 1.27 1.27)) (justify left))
@@
         )
       )
-    )
-  )
-  (symbol (lib_id "Device:R") (at 252.73 111.125 0) (unit 1)
-    (in_bom no) (on_board yes) (dnp yes) (fields_autoplaced)
-    (property "Reference" "R9" (at 255.27 110.49 0)
-      (effects (font (size 1.27 1.27)) (justify left))
-    )
-    (property "Value" "10k" (at 255.27 113.03 0)
-      (effects (font (size 1.27 1.27)) (justify left))
-    )
-    (property "Footprint" "Resistor_SMD:R_0603_1608Metric" (at 250.952 111.125 90)
-      (effects (font (size 1.27 1.27)) hide)
-    )
-    (property "Datasheet" "~" (at 252.73 111.125 0)
-      (effects (font (size 1.27 1.27)) hide)
-    )
-    (property "DPN" "1292-WR06X103JTLCT-ND" (at 252.73 111.125 0)
-      (effects (font (size 1.27 1.27)) hide)
-    )
-    (pin "1")
-    (pin "2")
-    (instances
-      (project "daq-wireless"
-        (path "/d87b4a87-5883-4edc-9ed5-8b7902b6705b"
-          (reference "R9") (unit 1)
-        )
-      )
