File: backplane-concept/backplane-concept.kicad_pcb (KiCad board)
At the start: 2 copper layers, 90 x 155.2 mm, 106 parts, among them J1 6473427-1, J2 PCIE_8x_Labeled, J3 PCIE_8x_Labeled, J4 PCIE_8x_Labeled, J5 CONN_MINI, J6 CONN_MINI, J7 CONN_MINI, J8 CONN_MINI, U1 PRIMARY, U2 SECONDARY, U3 NAU7802SGI, U4 ATA6561-GBQW-N, U5 ESP32-PICO-D4, U6 5V Reg, U7 AMS1117CD-5.0, U8 3.3V Reg, U9 AMS1117CD-3.3

Commit message: more roting
Parts:
- removed the TP42 at (153.8, 21.8)
- removed the TP42 at (153.0, 29.0)
- removed the TP42 at (150.5, 25.0)
- removed the TP42 at (150.2, 29.0)
- removed the TP42 at (153.2, 25.0)
- removed U4: ATA6561-GBQW-N, !footprints:ATA6561-GBQW-N
- removed U5: ESP32-PICO-D4, Package_DFN_QFN:QFN-48-1EP_7x7mm_P0.5mm_EP5.3x5.3mm
- added C27: 22uF, Capacitor_SMD:C_1210_3225Metric, F.Cu at (172.3, 123.0)
- added C28: 0.1uF, Capacitor_SMD:C_0603_1608Metric, F.Cu at (27.0, 149.2)
- added C29: 0.1uF, Capacitor_SMD:C_0603_1608Metric, F.Cu at (27.0, 156.7)
- added C30: 0.1uF, Capacitor_SMD:C_0603_1608Metric, F.Cu at (2.80, 155.6)
- added C31: 0.1uF, Capacitor_SMD:C_0603_1608Metric, F.Cu at (13.0, 147.0)
- added D1: 3V3A, LED_SMD:LED_0603_1608Metric, F.Cu at (167.4, 122.2)
- added D2: 5VA, LED_SMD:LED_0603_1608Metric, F.Cu at (167.4, 124.8)
- added D3: 5V, LED_SMD:LED_0603_1608Metric, F.Cu at (167.4, 127.3)
- added D4: 3V3, LED_SMD:LED_0603_1608Metric, F.Cu at (167.4, 129.9)
- added IC1: ISO6760DWR, !footprints:SOIC127P1030X265-16N, F.Cu at (20.7, 153.7)
- added IC2: ISO6760DWR, !footprints:SOIC127P1030X265-16N, F.Cu at (9.30, 153.7)
- added J10: ~, !footprints:5-5530843-3-EDGE, B.Cu at (51.0, 160.0)
- added J11: 1-967657-1, !footprints:19676571, F.Cu at (90.0, 43.4)
- added J9: POWER, Connector_PinHeader_2.54mm:PinHeader_1x05_P2.54mm_Vertical, F.Cu at (2.70, 3.52)
- added JP10: SolderJumper_2_Open, !footprints:JMP_Small, F.Cu at (10.9, 153.7)
- added JP11: SolderJumper_2_Open, !footprints:JMP_Small, F.Cu at (9.30, 153.7)
- added JP12: SolderJumper_2_Open, !footprints:JMP_Small, F.Cu at (7.71, 153.7)
- added JP2: SolderJumper_2_Open, !footprints:JMP_Small, F.Cu at (24.8, 153.6)
- added JP3: SolderJumper_2_Open, !footprints:JMP_Small, F.Cu at (23.2, 153.6)
- added JP4: SolderJumper_2_Open, !footprints:JMP_Small, F.Cu at (21.6, 153.6)
- added JP5: SolderJumper_2_Open, !footprints:JMP_Small, F.Cu at (20.0, 153.6)
- added JP6: SolderJumper_2_Open, !footprints:JMP_Small, F.Cu at (18.4, 153.6)
- added JP7: SolderJumper_2_Open, !footprints:JMP_Small, F.Cu at (16.8, 153.6)
- added JP8: SolderJumper_2_Open, !footprints:JMP_Small, F.Cu at (6.11, 153.7)
- added JP9: SolderJumper_2_Open, !footprints:JMP_Small, F.Cu at (12.5, 153.7)
- added R11: 120, Resistor_SMD:R_0603_1608Metric, F.Cu at (159.8, 65.7)
- added R12: 130, Resistor_SMD:R_0603_1608Metric, F.Cu at (159.8, 68.2)
- added R13: 300, Resistor_SMD:R_0603_1608Metric, F.Cu at (159.8, 70.7)
- added R14: 300, Resistor_SMD:R_0603_1608Metric, F.Cu at (159.8, 73.2)
- added R15: 130, Resistor_SMD:R_0603_1608Metric, F.Cu at (159.8, 75.8)
- C10, C12, C14, C15, C18, C23, C24, C7, C8, C9: footprint Capacitor_SMD:C_0805_2012Metric -> Capacitor_SMD:C_1210_3225Metric
- J1: value 6473427-1 -> ECVT I/O
- moved C7 153.9 mm to (31.5, 108.8), turned to -90 degrees
- moved C9 150.8 mm to (31.2, 99.1), turned to -90 degrees
- moved C10 149.7 mm to (31.2, 94.3), turned to -90 degrees
- moved U3 145.1 mm to (74.0, 71.7)
- moved C8 138.2 mm to (46.8, 107.8), turned to -90 degrees
- moved TP3 104.1 mm to (155.0, 28.9)
- moved TP4 104.1 mm to (155.0, 32.5)
- moved TP5 104.1 mm to (155.0, 36.0)
- moved TP1 101.8 mm to (151.5, 37.8)
- moved TP2 101.8 mm to (155.0, 40.8)
- moved TP6 101.8 mm to (155.2, 44.0)
- moved U7 98.2 mm to (39.7, 106.8), turned to 0 degrees
- moved U9 83.0 mm to (39.6, 96.3), turned to 0 degrees
- moved TP19 81.9 mm to (175.8, 47.0)
- moved TP22 81.9 mm to (179.0, 47.2)
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Connections:
- C10 pad 1: /PSU/3V3_CLEAN -> +3.3VA
- C12 pad 1: /PSU/VIN -> +8V
- C14 pad 1: /PSU/5V_HP -> +5V
- C15 pad 1: /PSU/5V_HP -> +5V
- C18 pad 1: /PSU/VIN -> +8V
- C23 pad 1: /PSU/3V3_HP -> +3V3
- C24 pad 1: /PSU/3V3_HP -> +3V3
- C25 pad 1: /PSU/VIN -> +8V
- C26 pad 1: /PSU/VIN -> +8V
- C7 pad 1: /PSU/VIN -> +8V
- C8 pad 1: /PSU/5V_CLEAN -> +5VA
- C9 pad 1: /PSU/VIN -> +8V
- J1 pad A10: +5V -> +5VA
- L1 pad 2: /PSU/5V_HP -> +5V
- L2 pad 2: /PSU/3V3_HP -> +3V3
- R6 pad 1: /PSU/5V_HP -> +5V
- R9 pad 1: /PSU/3V3_HP -> +3V3
- TP10 pad 1: /PSU/5V_HP -> +5V
- TP11 pad 1: /PSU/VIN -> +8V
- TP42 pad 1: (no net) -> I2C0_ECVT_SDA
- TP7 pad 1: /PSU/5V_CLEAN -> +5VA
- TP8 pad 1: /PSU/3V3_CLEAN -> +3.3VA
- TP9 pad 1: /PSU/3V3_HP -> +3V3
- U6 pad 2: /PSU/VIN -> +8V
- U6 pad 3: /PSU/VIN -> +8V
- U7 pad 2: /PSU/5V_CLEAN -> +5VA
- U7 pad 3: /PSU/VIN -> +8V
- U8 pad 2: /PSU/VIN -> +8V
- U8 pad 3: /PSU/VIN -> +8V
- U9 pad 2: /PSU/3V3_CLEAN -> +3.3VA
- U9 pad 3: /PSU/VIN -> +8V
Routing:
- net HALL3_S: track 0.00 -> 137.6 mm, vias 0 -> 2
- net HALL3_P: track 0.00 -> 122.4 mm, vias 0 -> 2
- net HALL1_S: track 0.00 -> 104.5 mm, vias 0 -> 2
- net ~ENCI_P: track 42.2 -> 145.5 mm, vias 0 -> 1
- net GND: track 523.6 -> 625.2 mm, vias 88 -> 103
- net HALL2_S: track 0.00 -> 100.9 mm, vias 0 -> 2
- net I2C0_ECVT_SCL: track 239.5 -> 138.9 mm, vias 23 -> 13
- net HALL1_P: track 0.00 -> 100.4 mm, vias 0 -> 2
- net HALL2_P: track 0.00 -> 99.4 mm, vias 0 -> 2
- net CAN_L: track 242.5 -> 143.7 mm, vias 23 -> 13
- net ENCI_P: track 47.9 -> 145.6 mm, vias 0 -> 1
- net I2C0_DAQ_SCL: track 243.9 -> 147.0 mm, vias 23 -> 13
- net ~ENCB_P: track 42.2 -> 138.7 mm, vias 0 -> 1
- net ENCI_S: track 46.9 -> 141.6 mm, vias 0 -> 1
- net ~ENCI_S: track 40.9 -> 135.3 mm, vias 0 -> 1
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Other:
- board size 90 x 155.2 mm -> 90 x 160 mm
- board text added: "ISO1 Bypass"
- board text added: "ISO2 Bypass"
- board text added: "Note: This dim is clearence from MATING connector to this board's edge."
- board text removed: "PSU Gen here"
- board text removed: "Single Flip"
- board text removed: "Single Rotation"
- board text removed: "Single Rotation (Center-Aligned)"
