File: backplane-concept/backplane-concept.kicad_pcb (KiCad board)
At the start: 2 copper layers, 90 x 160 mm, 129 parts, among them IC1 ISO6760DWR, IC2 ISO6760DWR, J1 ECVT I/O, J11 1-967657-1, J2 PCIE_8x_Labeled, J3 PCIE_8x_Labeled, J4 PCIE_8x_Labeled, J5 CONN_MINI, J6 CONN_MINI, J7 CONN_MINI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

Commit message: Moar Routing
Parts:
- removed C30: 0.1uF, Capacitor_SMD:C_0603_1608Metric
- removed J9: POWER, Connector_PinHeader_2.54mm:PinHeader_1x05_P2.54mm_Vertical
- removed R11: 120, Resistor_SMD:R_0603_1608Metric
- added J12: POWER, Connector_PinHeader_2.54mm:PinHeader_1x04_P2.54mm_Vertical, F.Cu at (2.60, 3.00)
- added JP1: AVDD_P, Jumper:SolderJumper-2_P1.3mm_Bridged_RoundedPad1.0x1.5mm, F.Cu at (83.9, 59.3)
- added JP13: AVDD_S, Jumper:SolderJumper-2_P1.3mm_Bridged_RoundedPad1.0x1.5mm, F.Cu at (81.2, 59.3)
- moved R15 143.2 mm to (29.5, 135.2), turned to 90 degrees
- moved TP11 140.3 mm to (27.6, -40.6)
- moved TP7 140.3 mm to (28.1, -36.8)
- moved TP8 140.3 mm to (28.1, -33.2)
- moved D4 138.0 mm to (29.5, 132.1), turned to -90 degrees
- moved C27 131.4 mm to (86.6, 23.4), turned to 90 degrees
- moved R14 130.5 mm to (45.0, 135.2), turned to 90 degrees
- moved D1 129.4 mm to (39.4, 103.7), turned to 90 degrees
- moved TP20 127.7 mm to (69.5, -31.9)
- moved TP14 127.7 mm to (81.5, -37.5)
- moved TP16 127.7 mm to (79.5, -33.8)
- moved TP19 127.7 mm to (67.5, -20.8)
- moved TP21 127.7 mm to (66.0, -31.9)
- moved TP22 127.7 mm to (70.8, -20.5)
- moved TP42 127.7 mm to (78.8, -25.8)
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Connections:
- C2 pad 1: AVDD_P -> Net-(JP1-B)
- C3 pad 1: AVDD_P -> Net-(JP1-B)
- J1 pad B22: AVDD_P -> AVDD_S
- J2 pad B30: LOADC_CLK_P -> LOADC_CLK_S
- J3 pad B30: LOADC_CLK_P -> LOADC_CLK_S
- J4 pad B30: LOADC_CLK_P -> LOADC_CLK_S
- TP5 pad 1: AVDD_P -> AVDD_S
- U2 pad 1: AVDD_P -> AVDD_S
- U2 pad 10: +5V -> +5VA
- U3 pad 1: AVDD_P -> Net-(JP1-B)
- U3 pad 16: AVDD_P -> Net-(JP1-B)
Routing:
- net +5VA: track 13.3 -> 207.2 mm, vias 0 -> 15
- net +3.3VA: track 14.5 -> 159.2 mm, vias 0 -> 5
- net +8V: track 26.5 -> 157.7 mm, vias 26 -> 33
- net DIR_P: track 82.4 -> 198.3 mm, vias 7 -> 8
- net PWM_P: track 83.4 -> 199.0 mm, vias 7 -> 8
- net CAN_H: track 134.8 -> 250.3 mm, vias 13 -> 14
- net PWM_S: track 113.4 -> 227.6 mm, vias 10 -> 11
- net DIR_S: track 85.3 -> 199.3 mm, vias 7 -> 8
- net CAN_L: track 143.7 -> 255.6 mm, vias 13 -> 14
- net LOADC_CLK_S: track 0.00 -> 101.0 mm, vias 0 -> 6
- net AVDD_S: track 0.00 -> 82.9 mm, vias 0 -> 1
- net AVDD_P: track 11.0 -> 91.2 mm, vias 0 -> 1
- net THERM_S: track 61.4 -> 129.1 mm
- net THERM_P: track 78.0 -> 141.2 mm
- net IN-_S: track 4.45 -> 62.7 mm, vias 0 -> 2
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
Commit message: Finish Routing
Parts:
- removed TP10: 5VHP, !footprints:TestPoint_Pad_D1.0mm
- removed TP11: VIN, !footprints:TestPoint_Pad_D1.0mm
- removed TP7: 5VC, !footprints:TestPoint_Pad_D1.0mm
- removed TP8: 3V3C, !footprints:TestPoint_Pad_D1.0mm
- removed TP9: 3V3HP, !footprints:TestPoint_Pad_D1.0mm
- moved TP42 65.8 mm to (20.8, 5.25)
- moved TP14 65.4 mm to (48.2, 18.8), turned to -60 degrees
- moved TP15 62.9 mm to (49.8, 18.8), turned to -60 degrees
- moved TP43 61.9 mm to (22.2, 5.25)
- moved TP16 59.6 mm to (51.2, 18.8), turned to -60 degrees
- moved TP17 57.4 mm to (52.8, 18.8), turned to -60 degrees
- moved TP20 46.6 mm to (41.3, 5.30)
- moved TP21 43.8 mm to (42.8, 5.30)
- moved TP19 38.1 mm to (39.8, 5.30)
- moved TP22 37.0 mm to (44.3, 5.30)
Connections:
- J2 pad B48: Net-(J2-PadB48) -> ADC_IRQ
- J3 pad B48: Net-(J2-PadB48) -> ADC_IRQ
- J4 pad B48: Net-(J2-PadB48) -> ADC_IRQ
- U3 pad 12: /Analog Frontend/IRQ -> ADC_IRQ
- U3 pad 13: /Analog Frontend/SCL -> I2C0_ECVT_SCL
- U3 pad 14: /Analog Frontend/SDA -> I2C0_ECVT_SDA
Routing:
- net ADC_IRQ: track 0.00 -> 80.4 mm, vias 0 -> 7
- net I2C0_ECVT_SCL: track 138.9 -> 197.6 mm
- net I2C0_ECVT_SDA: track 132.2 -> 190.8 mm
- net Net-(J2-PadB48): track 53.2 -> 0.00 mm, vias 5 -> 0
- net RPOT2: track 91.1 -> 43.9 mm, vias 9 -> 4
- net LOADC_DAT_P: track 147.1 -> 113.0 mm, vias 10 -> 6
- net I2C1_ECVT_EXT_SDA: track 141.9 -> 107.9 mm, vias 11 -> 7
- net Net-(J2-PadB49): track 85.5 -> 53.0 mm, vias 7 -> 4
- net HALL_ENG1: track 151.3 -> 120.7 mm, vias 11 -> 8
- net GND: track 604.7 -> 579.4 mm, vias 121 -> 119
- net PWM_S: track 227.6 -> 202.8 mm, vias 11 -> 7
- net LOADC_DAT_S: track 106.1 -> 85.1 mm, vias 6 -> 4
- net LOADC_CLK_S: track 101.0 -> 80.7 mm, vias 6 -> 4
- net BP_REAR: track 63.4 -> 44.3 mm, vias 6 -> 4
- net LOADC_CLK_P: track 126.4 -> 107.4 mm, vias 6 -> 4
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
Commit message: TODO
Holes,
double check
Other:
- board text added: "Backplane Concept V1.1 Designed by D.C."
Changed lines of the file:
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@@
     (effects (font (size 0.75 0.75) (thickness 0.09375)) (justify left bottom))
+  )
+  (gr_text "Backplane Concept V1.1\nDesigned by D.C." (at 70 158.25) (layer "F.SilkS")
+    (effects (font (size 1 1) (thickness 0.15)) (justify left bottom))
   )
   (gr_text "PSU Interconnect here\n" (at 13 158.25) (layer "Cmts.User")
