File: backplane-concept/analog_frontend.kicad_sch (KiCad schematic)
At the start: 13 parts, among them U1 PRIMARY, U2 SECONDARY, U3 NAU7802SGI

Commit message: Design PSUs, route bucks
Parts:
- C1, C2, C3, C4, C5, C6: footprint (none) -> Capacitor_SMD:C_0603_1608Metric
- R1, R2, R3, R4: footprint (none) -> Resistor_SMD:R_0603_1608Metric
- U1, U2: footprint SPARKFUN_SEN-13879 -> !footprints:SPARKFUN_SEN-13879
Connections:
- net +5V: no longer U1.10 (VDD)
- net +3V3 renamed +3.3VA
- new net +5VA: U1.10 (VDD)

Commit message: more roting
Parts:
- U3: DPN (none) -> NAU7802SGI-ND
Changed lines of the file:
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@@
       (effects (font (size 1.524 1.524)) hide)
+    )
+    (property "DPN" "NAU7802SGI-ND" (at 158.75 97.155 0)
+      (effects (font (size 1.27 1.27)) hide)
     )
     (pin "1")

Commit message: Moar Routing
Parts:
- added JP1: AVDD_P, Jumper:SolderJumper-2_P1.3mm_Bridged_RoundedPad1.0x1.5mm, symbol Jumper:SolderJumper_2_Bridged
- added JP13: AVDD_S, Jumper:SolderJumper-2_P1.3mm_Bridged_RoundedPad1.0x1.5mm, symbol Jumper:SolderJumper_2_Bridged
Connections:
- net +5V is gone; now on net +5VA: U2.10 (VDD)
- net AVDD_P: now also JP1.1 (A); no longer C2.1, C3.1, U2.1 (RED), U3.1 (REFP), U3.16 (AVDD/LDO)
- new net: C2.1, C3.1, JP1.2 (B), JP13.2 (B), U3.1 (REFP), U3.16 (AVDD/LDO)
- new net AVDD_S: JP13.1 (A), U2.1 (RED)
Changed lines of the file:
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@@
   (junction (at 146.05 82.55) (diameter 0) (color 0 0 0 0)
+  )
+  (junction (at 127 82.55) (diameter 0) (color 0 0 0 0)
   )
   (junction (at 209.55 124.46) (diameter 0) (color 0 0 0 0)
@@
     (stroke (width 0) (type default))
   )
-  (wire (pts (xy 127 82.55) (xy 127 84.455))
+  (wire (pts (xy 127 82.55) (xy 127 85.725))
     (stroke (width 0) (type default))
   )
@@
     (effects (font (size 1.27 1.27)) (justify left))
   )
-  (hierarchical_label "AVDD_P" (shape input) (at 127 82.55 180) (fields_autoplaced)
+  (hierarchical_label "AVDD_S" (shape input) (at 119.38 85.725 180) (fields_autoplaced)
     (effects (font (size 1.27 1.27)) (justify right))
   )
@@
     (effects (font (size 1.27 1.27)) (justify left))
   )
-  (hierarchical_label "AVDD_S" (shape input) (at 127 84.455 180) (fields_autoplaced)
+  (hierarchical_label "AVDD_P" (shape input) (at 119.38 82.55 180) (fields_autoplaced)
     (effects (font (size 1.27 1.27)) (justify right))
   )
@@
     )
   )
+  (symbol (lib_id "Jumper:SolderJumper_2_Bridged") (at 123.19 82.55 0) (unit 1)
+    (in_bom yes) (on_board yes) (dnp no) (fields_autoplaced)
+    (property "Reference" "JP1" (at 123.19 77.47 0)
+      (effects (font (size 1.27 1.27)))
+    )
+    (property "Value" "AVDD_P" (at 123.19 80.01 0)
+      (effects (font (size 1.27 1.27)))
+    )
+    (property "Footprint" "Jumper:SolderJumper-2_P1.3mm_Bridged_RoundedPad1.0x1.5mm" (at 123.19 82.55 0)
+      (effects (font (size 1.27 1.27)) hide)
+    )
+    (property "Datasheet" "~" (at 123.19 82.55 0)
+      (effects (font (size 1.27 1.27)) hide)
+    )
+    (pin "1")
+    (pin "2")
+    (instances
+      (project "backplane-concept"
+        (path "/1eedfbfd-a1b6-445d-9b0a-8fd3d481d4f1/288bfc7c-fd6f-4456-8ab8-dbe85b450aa5"
+          (reference "JP1") (unit 1)
+        )
+      )
+    )
+  )
   (symbol (lib_id "Device:C") (at 134.62 100.965 0) (unit 1)
     (in_bom yes) (on_board yes) (dnp no)
@@
     )
   )
+  (symbol (lib_id "Jumper:SolderJumper_2_Bridged") (at 123.19 85.725 0) (unit 1)
+    (in_bom yes) (on_board yes) (dnp no) (fields_autoplaced)
+    (property "Reference" "JP13" (at 123.19 81.28 0)
+      (effects (font (size 1.27 1.27)))
+    )
+    (property "Value" "AVDD_S" (at 123.19 83.82 0)
+      (effects (font (size 1.27 1.27)))
+    )
+    (property "Footprint" "Jumper:SolderJumper-2_P1.3mm_Bridged_RoundedPad1.0x1.5mm" (at 123.19 85.725 0)
+      (effects (font (size 1.27 1.27)) hide)
+    )
+    (property "Datasheet" "~" (at 123.19 85.725 0)
+      (effects (font (size 1.27 1.27)) hide)
+    )
+    (pin "1")
+    (pin "2")
+    (instances
+      (project "backplane-concept"
+        (path "/1eedfbfd-a1b6-445d-9b0a-8fd3d481d4f1/288bfc7c-fd6f-4456-8ab8-dbe85b450aa5"
+          (reference "JP13") (unit 1)
+        )
+      )
+    )
+  )
   (symbol (lib_id "power:GND") (at 213.36 90.17 0) (unit 1)
     (in_bom yes) (on_board yes) (dnp no) (fields_autoplaced)
@@
         (path "/1eedfbfd-a1b6-445d-9b0a-8fd3d481d4f1/288bfc7c-fd6f-4456-8ab8-dbe85b450aa5"
           (reference "#PWR013") (unit 1)
-        )
-      )
-    )
-  )
-  (symbol (lib_id "power:+5V") (at 78.74 114.935 0) (unit 1)
-    (in_bom yes) (on_board yes) (dnp no) (fields_autoplaced)
-    (property "Reference" "#PWR07" (at 78.74 118.745 0)
-      (effects (font (size 1.27 1.27)) hide)
-    )
-    (property "Value" "+5V" (at 78.74 111.76 0)
-      (effects (font (size 1.27 1.27)))
-    )
-    (property "Footprint" "" (at 78.74 114.935 0)
-      (effects (font (size 1.27 1.27)) hide)
-    )
-    (property "Datasheet" "" (at 78.74 114.935 0)
-      (effects (font (size 1.27 1.27)) hide)
-    )
-    (pin "1")
-    (instances
-      (project "backplane-concept"
-        (path "/1eedfbfd-a1b6-445d-9b0a-8fd3d481d4f1/288bfc7c-fd6f-4456-8ab8-dbe85b450aa5"
-          (reference "#PWR07") (unit 1)
         )
       )
@@
         )
       )
+    )
+  )
+  (symbol (lib_id "power:+5VA") (at 78.74 114.935 0) (unit 1)
+    (in_bom yes) (on_board yes) (dnp no) (fields_autoplaced)
+    (property "Reference" "#PWR065" (at 78.74 118.745 0)
+      (effects (font (size 1.27 1.27)) hide)
+    )
+    (property "Value" "+5VA" (at 78.74 111.76 0)
+      (effects (font (size 1.27 1.27)))
+    )
+    (property "Footprint" "" (at 78.74 114.935 0)
+      (effects (font (size 1.27 1.27)) hide)
+    )
+    (property "Datasheet" "" (at 78.74 114.935 0)
+      (effects (font (size 1.27 1.27)) hide)
+    )
+    (pin "1")
+    (instances
+      (project "backplane-concept"
+        (path "/1eedfbfd-a1b6-445d-9b0a-8fd3d481d4f1/288bfc7c-fd6f-4456-8ab8-dbe85b450aa5"
+          (reference "#PWR065") (unit 1)
+        )
+      )
