File: backplane-concept/backplane-concept.kicad_sch (KiCad schematic)
At the start: 51 parts, among them J1 6473427-1, J2 PCIE_8x_Labeled, J3 PCIE_8x_Labeled, J4 PCIE_8x_Labeled, J5 CONN_MINI, J6 CONN_MINI, J7 CONN_MINI, J8 CONN_MINI, U4 ATA6561-GBQW-N, U5 ESP32-PICO-D4

Commit message: more roting
Parts:
- removed U4: ATA6561-GBQW-N, !footprints:ATA6561-GBQW-N, symbol ATA6561:ATA6561-GBQW-N
- removed U5: ESP32-PICO-D4, Package_DFN_QFN:QFN-48-1EP_7x7mm_P0.5mm_EP5.3x5.3mm, symbol RF_Module:ESP32-PICO-D4
- added C27: 22uF, Capacitor_SMD:C_1210_3225Metric, symbol Device:C
- added C28, C29, C30, C31: 0.1uF, Capacitor_SMD:C_0603_1608Metric, symbol Device:C
- added D1: 3V3A, LED_SMD:LED_0603_1608Metric, symbol Device:D
- added D2: 5VA, LED_SMD:LED_0603_1608Metric, symbol Device:D
- added D3: 5V, LED_SMD:LED_0603_1608Metric, symbol Device:D
- added D4: 3V3, LED_SMD:LED_0603_1608Metric, symbol Device:D
- added IC1, IC2: ISO6760DWR, !footprints:SOIC127P1030X265-16N, symbol ISO6760DWR:ISO6760DWR
- added J10: ~, !footprints:5-5530843-3-EDGE, symbol !CUSTOM:Powerboard_Conn
- added J11: 1-967657-1, !footprints:19676571, symbol 1-967657-1:1-967657-1
- added J9: POWER, Connector_PinHeader_2.54mm:PinHeader_1x05_P2.54mm_Vertical, symbol Connector:Conn_01x05_Pin
- added JP10, JP11, JP12, JP2, JP3, JP4, JP5, JP6, JP7, JP8, JP9: SolderJumper_2_Open, !footprints:JMP_Small, symbol Jumper:SolderJumper_2_Open
- added R11: 120, Resistor_SMD:R_0603_1608Metric, symbol Device:R
- added R12, R15: 130, Resistor_SMD:R_0603_1608Metric, symbol Device:R
- added R13, R14: 300, Resistor_SMD:R_0603_1608Metric, symbol Device:R
- J1: value 6473427-1 -> ECVT I/O
- J2, J3, J4: DPN (none) -> A109484-ND
- J5, J6, J7, J8: DPN (none) -> 609-2025-ND
Connections:
- net +3.3VA: now also J9.5 (Pin_5), R12.1
- net +3V3: now also J9.3 (Pin_3), R15.1
- net +5V: now also J9.2 (Pin_2), R14.1; no longer J1.A10
- net +5VA: now also J1.A10, C28.1, C31.1, IC1.1 (VCC1), IC2.1 (VCC1), J9.4 (Pin_4), R13.1
- net +8V: now also C27.1, J11.2 (VBATT)
- net CAN_H: now also J10.B17 (CANH), J11.4 (CANH), R11.1
- net CAN_L: now also J10.A17 (CANL), J11.3 (CANL), R11.2
- net DIR_P: now also IC2.3 (INB), JP10.1 (A)
- net DIR_S: now also IC2.5 (IND), JP12.1 (A)
- net GND: now also C27.2, C28.2, C31.2, D1.1 (K), D2.1 (K), D3.1 (K), D4.1 (K), IC1.8 (GND1), IC2.8 (GND1), J11.1 (GND), J9.1 (Pin_1), JP8.1 (A)
- net HALL1_P: now also IC1.2 (INA), JP2.1 (A)
- net HALL1_S: now also IC1.5 (IND), JP5.1 (A)
- net HALL2_P: now also IC1.3 (INB), JP3.1 (A)
- net HALL2_S: now also IC1.6 (INE), JP6.1 (A)
- net HALL3_P: now also IC1.4 (INC), JP4.1 (A)
- net HALL3_S: now also IC1.7 (INF), JP7.1 (A)
- net MOT1_P: now also J10.A1 (MOT1_P), J10.A2, J10.A3
- net MOT1_S: now also J10.B7 (MOT3_S), J10.B8, J10.B9
- net MOT2_P: now also J10.A4 (MOT2_P), J10.A5, J10.A6
- net MOT2_S: now also J10.B4 (MOT2_S), J10.B5, J10.B6 (MOT3_S)
- net MOT3_P: now also J10.A7 (MOT3_P), J10.A8, J10.A9
- net MOT3_S: now also J10.B1 (MOT1_S), J10.B2, J10.B3
- net PWM_P: now also IC2.2 (INA), JP9.1 (A)
- net PWM_S: now also IC2.4 (INC), JP11.1 (A)
- new net: D1.2 (A), R12.2
- new net: D4.2 (A), R15.2
- new net: D2.2 (A), R13.2
- new net: D3.2 (A), R14.2
- new net DIR_P_ISO: IC2.14 (OUTB), J10.A15 (PWM_P), JP10.2 (B)
- new net DIR_S_ISO: IC2.12 (OUTD), J10.B15 (PWM_S), JP12.2 (B)
- new net HALL1_P_ISO: IC1.15 (OUTA), J10.A11 (HALL1_P), JP2.2 (B)
- new net HALL1_S_ISO: IC1.12 (OUTD), J10.B11 (HALL1_S), JP5.2 (B)
- new net HALL2_P_ISO: IC1.14 (OUTB), J10.A12 (HALL2_P), JP3.2 (B)
- new net HALL2_S_ISO: IC1.11 (OUTE), J10.B12 (HALL2_S), JP6.2 (B)
- new net HALL3_P_ISO: IC1.13 (OUTC), J10.A13 (HALL3_P), JP4.2 (B)
- new net HALL3_S_ISO: IC1.10 (OUTF), J10.B13 (HALL3_S), JP7.2 (B)
- new net PWM_P_ISO: IC2.15 (OUTA), J10.A14 (DIR_P), JP9.2 (B)
- new net PWM_S_ISO: IC2.13 (OUTC), J10.B14 (DIR_S), JP11.2 (B)
- new net VDD_ISO: C29.1, C30.1, IC1.16 (VCC2), IC2.16 (VCC2), J10.A10 (VDD), J10.B10 (VDD)
- new net VSS_ISO: C29.2, C30.2, IC1.9 (GND2), IC2.9 (GND2), J10.A16 (VSS), J10.B16 (VSS), JP8.2 (B)
- no-connect marks 0 -> 4
Other:
- sheet PSU ports: added 3V3_CLEAN, 3V3_HP, 5V_CLEAN, 5V_HP, VIN; removed none
- note added: "ISO 1 Bypass"
- note added: "ISO 2 Bypass"
- note added: "NOTE: Only install at CAN Termination!"
- note added: "Note: Reversal here makes routing easier. It won't affect performance"
- note added: "TODO - Add CAN/DAQ sealable connector - Battery Conn, Position"
- moved on the sheet: J1, J2, J3, J4, J5, J6, J7, J8

Commit message: Moar Routing
Parts:
- removed C30: 0.1uF, Capacitor_SMD:C_0603_1608Metric, symbol Device:C
- removed J9: POWER, Connector_PinHeader_2.54mm:PinHeader_1x05_P2.54mm_Vertical, symbol Connector:Conn_01x05_Pin
- removed R11: 120, Resistor_SMD:R_0603_1608Metric, symbol Device:R
- added J12: POWER, Connector_PinHeader_2.54mm:PinHeader_1x04_P2.54mm_Vertical, symbol Connector:Conn_01x04_Pin
Connections:
- net +3V3: now also J12.3 (Pin_3)
- net +5V: now also J12.2 (Pin_2)
- net +8V: now also J12.4 (Pin_4)
- net GND: now also J12.1 (Pin_1)
- net LOADC_CLK_P: no longer J2.B30 (LOADC_CLK_S), J3.B30 (LOADC_CLK_S), J4.B30 (LOADC_CLK_S)
- net LOADC_CLK_S: now also J2.B30 (LOADC_CLK_S), J3.B30 (LOADC_CLK_S), J4.B30 (LOADC_CLK_S)
Other:
- note removed: "NOTE: Only install at CAN Termination!"

Commit message: Finish Routing
Connections:
- net ADC_IRQ: now reaches J2.B48, J3.B48, J4.B48
Changed lines of the file:
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@@
+    (stroke (width 0) (type default))
+  )
+  (wire (pts (xy 326.39 34.29) (xy 330.2 34.29))
     (stroke (width 0) (type default))
   )
@@
     (stroke (width 0) (type default))
   )
+  (wire (pts (xy 96.52 149.225) (xy 107.315 149.225))
+    (stroke (width 0) (type default))
+  )
   (wire (pts (xy 107.315 100.965) (xy 96.52 100.965))
     (stroke (width 0) (type default))
@@
     (stroke (width 0) (type default))
   )
+  (wire (pts (xy 326.39 36.83) (xy 330.2 36.83))
+    (stroke (width 0) (type default))
+  )
   (wire (pts (xy 36.195 121.285) (xy 38.1 121.285))
     (stroke (width 0) (type default))
@@
   )
   (wire (pts (xy 107.315 113.665) (xy 98.425 113.665))
+    (stroke (width 0) (type default))
+  )
+  (wire (pts (xy 326.39 31.75) (xy 330.2 31.75))
     (stroke (width 0) (type default))
   )
@@
     )
   )
+  (global_label "ADC_IRQ" (shape passive) (at 330.2 36.83 0) (fields_autoplaced)
+    (effects (font (size 1.27 1.27)) (justify left))
+    (property "Intersheetrefs" "${INTERSHEET_REFS}" (at 339.796 36.83 0)
+      (effects (font (size 1.27 1.27)) (justify left) hide)
+    )
+  )
   (global_label "I2C0_ECVT_SDA" (shape passive) (at 107.315 52.705 0) (fields_autoplaced)
     (effects (font (size 1.27 1.27)) (justify left))
@@
     (property "Intersheetrefs" "${INTERSHEET_REFS}" (at 289.0052 57.15 0)
       (effects (font (size 1.27 1.27)) (justify right) hide)
+    )
+  )
+  (global_label "I2C0_ECVT_SCL" (shape passive) (at 330.2 31.75 0) (fields_autoplaced)
+    (effects (font (size 1.27 1.27)) (justify left))
+    (property "Intersheetrefs" "${INTERSHEET_REFS}" (at 346.2063 31.75 0)
+      (effects (font (size 1.27 1.27)) (justify left) hide)
     )
   )
@@
     )
   )
+  (global_label "ADC_IRQ" (shape passive) (at 107.315 149.225 0) (fields_autoplaced)
+    (effects (font (size 1.27 1.27)) (justify left))
+    (property "Intersheetrefs" "${INTERSHEET_REFS}" (at 116.911 149.225 0)
+      (effects (font (size 1.27 1.27)) (justify left) hide)
+    )
+  )
+  (global_label "I2C0_ECVT_SDA" (shape passive) (at 330.2 34.29 0) (fields_autoplaced)
+    (effects (font (size 1.27 1.27)) (justify left))
+    (property "Intersheetrefs" "${INTERSHEET_REFS}" (at 346.2668 34.29 0)
+      (effects (font (size 1.27 1.27)) (justify left) hide)
+    )
+  )
