File: backplane-concept/psu.kicad_sch (KiCad schematic)
At the start: 32 parts, among them U6 5V Reg, U6 AMS1117CD-5.0, U7 AMS1117CD-3.3, U8 3.3V Reg

Commit message: Add testpoints
Parts:
- added TP1: 3V3HP, !footprints:TestPoint_Pad_D1.0mm, symbol Connector:TestPoint_Small
- added TP1: 3V3C, !footprints:TestPoint_Pad_D1.0mm, symbol Connector:TestPoint_Small
- added TP1: VIN, !footprints:TestPoint_Pad_D1.0mm, symbol Connector:TestPoint_Small
- added TP1: 5VC, !footprints:TestPoint_Pad_D1.0mm, symbol Connector:TestPoint_Small
- added TP1: 5VHP, !footprints:TestPoint_Pad_D1.0mm, symbol Connector:TestPoint_Small
Connections:
- net +3.3VA renamed 3V3_CLEAN
- net 3V3_CLEAN: now also TP1.1
- net +3V3 renamed 3V3_HP
- net 3V3_HP: now also TP1.1
- net +5V renamed 5V_HP
- net 5V_HP: now also TP1.1
- net +5VA renamed 5V_CLEAN
- net 5V_CLEAN: now also TP1.1
- net +8V renamed VIN
- net VIN: now also TP1.1

Commit message: more roting
Parts:
- C10, C12, C14, C15, C18, C23, C24, C7, C8, C9: footprint Capacitor_SMD:C_0805_2012Metric -> Capacitor_SMD:C_1210_3225Metric; DPN (none) -> 1276-3395-1-ND
- U6: DPN (none) -> 4518-AMS1117CD-5.0CT-ND
- U7: DPN (none) -> 4518-AMS1117CD-3.3CT-ND
Changed lines of the file:
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@@
+      (effects (font (size 1.27 1.27)) hide)
+    )
+    (property "DPN" "4518-AMS1117CD-3.3CT-ND" (at 36.195 39.37 0)
       (effects (font (size 1.27 1.27)) hide)
     )
@@
       (effects (font (size 1.27 1.27)) (justify left))
     )
-    (property "Footprint" "Capacitor_SMD:C_0805_2012Metric" (at 113.9698 45.085 0)
+    (property "Footprint" "Capacitor_SMD:C_1210_3225Metric" (at 113.9698 45.085 0)
       (effects (font (size 1.27 1.27)) hide)
     )
@@
       (effects (font (size 1.27 1.27)) hide)
     )
+    (property "DPN" "1276-3395-1-ND" (at 114.935 41.275 0)
+      (effects (font (size 1.27 1.27)) hide)
+    )
     (pin "1")
     (pin "2")
@@
       (effects (font (size 1.27 1.27)) (justify left))
     )
-    (property "Footprint" "Capacitor_SMD:C_0805_2012Metric" (at 115.2398 113.03 0)
+    (property "Footprint" "Capacitor_SMD:C_1210_3225Metric" (at 115.2398 113.03 0)
       (effects (font (size 1.27 1.27)) hide)
     )
@@
       (effects (font (size 1.27 1.27)) hide)
     )
-    (property "DPN" "" (at 116.205 109.22 0)
+    (property "DPN" "1276-3395-1-ND" (at 116.205 109.22 0)
       (effects (font (size 1.27 1.27)) hide)
     )
@@
       (effects (font (size 1.27 1.27)) (justify left))
     )
-    (property "Footprint" "Capacitor_SMD:C_0805_2012Metric" (at 23.1902 46.99 0)
+    (property "Footprint" "Capacitor_SMD:C_1210_3225Metric" (at 23.1902 46.99 0)
       (effects (font (size 1.27 1.27)) hide)
     )
@@
       (effects (font (size 1.27 1.27)) hide)
     )
+    (property "DPN" "1276-3395-1-ND" (at 22.225 43.18 0)
+      (effects (font (size 1.27 1.27)) hide)
+    )
     (pin "1")
     (pin "2")
@@
       (effects (font (size 1.27 1.27)) (justify left))
     )
-    (property "Footprint" "Capacitor_SMD:C_0805_2012Metric" (at 213.6902 123.19 0)
+    (property "Footprint" "Capacitor_SMD:C_1210_3225Metric" (at 213.6902 123.19 0)
       (effects (font (size 1.27 1.27)) hide)
     )
@@
       (effects (font (size 1.27 1.27)) hide)
     )
-    (property "DPN" "" (at 212.725 119.38 0)
+    (property "DPN" "1276-3395-1-ND" (at 212.725 119.38 0)
       (effects (font (size 1.27 1.27)) hide)
     )
@@
       (effects (font (size 1.27 1.27)) (justify left))
     )
-    (property "Footprint" "Capacitor_SMD:C_0805_2012Metric" (at 25.7302 113.03 0)
+    (property "Footprint" "Capacitor_SMD:C_1210_3225Metric" (at 25.7302 113.03 0)
       (effects (font (size 1.27 1.27)) hide)
     )
@@
       (effects (font (size 1.27 1.27)) hide)
     )
+    (property "DPN" "1276-3395-1-ND" (at 24.765 109.22 0)
+      (effects (font (size 1.27 1.27)) hide)
+    )
     (pin "1")
     (pin "2")
@@
       (effects (font (size 1.27 1.27)) (justify left))
     )
-    (property "Footprint" "Capacitor_SMD:C_0805_2012Metric" (at 52.3748 113.03 0)
+    (property "Footprint" "Capacitor_SMD:C_1210_3225Metric" (at 52.3748 113.03 0)
       (effects (font (size 1.27 1.27)) hide)
     )
     (property "Datasheet" "~" (at 53.34 109.22 0)
+      (effects (font (size 1.27 1.27)) hide)
+    )
+    (property "DPN" "1276-3395-1-ND" (at 53.34 109.22 0)
       (effects (font (size 1.27 1.27)) hide)
     )
@@
       (effects (font (size 1.27 1.27)) (justify left))
     )
-    (property "Footprint" "Capacitor_SMD:C_0805_2012Metric" (at 220.0402 123.19 0)
+    (property "Footprint" "Capacitor_SMD:C_1210_3225Metric" (at 220.0402 123.19 0)
       (effects (font (size 1.27 1.27)) hide)
     )
@@
       (effects (font (size 1.27 1.27)) hide)
     )
-    (property "DPN" "" (at 219.075 119.38 0)
+    (property "DPN" "1276-3395-1-ND" (at 219.075 119.38 0)
       (effects (font (size 1.27 1.27)) hide)
     )
@@
     )
     (property "Datasheet" "http://www.advanced-monolithic.com/pdf/ds1117.pdf" (at 41.275 111.76 0)
+      (effects (font (size 1.27 1.27)) hide)
+    )
+    (property "DPN" "4518-AMS1117CD-5.0CT-ND" (at 38.735 105.41 0)
       (effects (font (size 1.27 1.27)) hide)
     )
@@
       (effects (font (size 1.27 1.27)) (justify left))
     )
-    (property "Footprint" "Capacitor_SMD:C_0805_2012Metric" (at 219.4052 55.245 0)
+    (property "Footprint" "Capacitor_SMD:C_1210_3225Metric" (at 219.4052 55.245 0)
       (effects (font (size 1.27 1.27)) hide)
     )
     (property "Datasheet" "~" (at 218.44 51.435 0)
+      (effects (font (size 1.27 1.27)) hide)
+    )
+    (property "DPN" "1276-3395-1-ND" (at 218.44 51.435 0)
       (effects (font (size 1.27 1.27)) hide)
     )
@@
       (effects (font (size 1.27 1.27)) (justify left))
     )
-    (property "Footprint" "Capacitor_SMD:C_0805_2012Metric" (at 49.8348 46.99 0)
+    (property "Footprint" "Capacitor_SMD:C_1210_3225Metric" (at 49.8348 46.99 0)
       (effects (font (size 1.27 1.27)) hide)
     )
@@
       (effects (font (size 1.27 1.27)) hide)
     )
+    (property "DPN" "1276-3395-1-ND" (at 50.8 43.18 0)
+      (effects (font (size 1.27 1.27)) hide)
+    )
     (pin "1")
     (pin "2")
@@
       (effects (font (size 1.27 1.27)) (justify left))
     )
-    (property "Footprint" "Capacitor_SMD:C_0805_2012Metric" (at 213.0552 55.245 0)
+    (property "Footprint" "Capacitor_SMD:C_1210_3225Metric" (at 213.0552 55.245 0)
       (effects (font (size 1.27 1.27)) hide)
     )
@@
       (effects (font (size 1.27 1.27)) hide)
     )
+    (property "DPN" "1276-3395-1-ND" (at 212.09 51.435 0)
+      (effects (font (size 1.27 1.27)) hide)
+    )

Commit message: TODO
Holes,
double check
Parts:
- removed TP1: 3V3HP, !footprints:TestPoint_Pad_D1.0mm, symbol Connector:TestPoint_Small
- removed TP1: 3V3C, !footprints:TestPoint_Pad_D1.0mm, symbol Connector:TestPoint_Small
- removed TP1: VIN, !footprints:TestPoint_Pad_D1.0mm, symbol Connector:TestPoint_Small
- removed TP1: 5VC, !footprints:TestPoint_Pad_D1.0mm, symbol Connector:TestPoint_Small
- removed TP1: 5VHP, !footprints:TestPoint_Pad_D1.0mm, symbol Connector:TestPoint_Small
Changed lines of the file:
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@@
-    (stroke (width 0) (type default))
-  )
-  (wire (pts (xy 34.29 140.97) (xy 37.465 140.97))
     (stroke (width 0) (type default))
   )
@@
     (stroke (width 0) (type default))
   )
-  (wire (pts (xy 34.29 154.305) (xy 37.465 154.305))
-    (stroke (width 0) (type default))
-  )
   (wire (pts (xy 36.195 46.99) (xy 50.8 46.99))
     (stroke (width 0) (type default))
@@
     (stroke (width 0) (type default))
   )
-  (wire (pts (xy 34.29 145.415) (xy 37.465 145.415))
-    (stroke (width 0) (type default))
-  )
   (wire (pts (xy 114.935 46.355) (xy 114.935 45.085))
     (stroke (width 0) (type default))
@@
     (stroke (width 0) (type default))
   )
-  (wire (pts (xy 34.29 149.86) (xy 37.465 149.86))
-    (stroke (width 0) (type default))
-  )
   (wire (pts (xy 20.955 105.41) (xy 24.765 105.41))
     (stroke (width 0) (type default))
@@
   )
   (wire (pts (xy 212.725 115.57) (xy 219.075 115.57))
-    (stroke (width 0) (type default))
-  )
-  (wire (pts (xy 34.29 158.75) (xy 37.465 158.75))
     (stroke (width 0) (type default))
   )
@@
     (effects (font (size 1.27 1.27)) (justify right))
   )
-  (hierarchical_label "3V3_CLEAN" (shape input) (at 34.29 149.86 180) (fields_autoplaced)
-    (effects (font (size 1.27 1.27)) (justify right))
-  )
   (hierarchical_label "VIN" (shape input) (at 116.205 102.87 90) (fields_autoplaced)
     (effects (font (size 1.27 1.27)) (justify left))
   )
-  (hierarchical_label "VIN" (shape input) (at 34.29 140.97 180) (fields_autoplaced)
-    (effects (font (size 1.27 1.27)) (justify right))
-  )
   (hierarchical_label "VIN" (shape input) (at 20.955 105.41 180) (fields_autoplaced)
     (effects (font (size 1.27 1.27)) (justify right))
@@
     (effects (font (size 1.27 1.27)) (justify left))
   )
-  (hierarchical_label "5V_HP" (shape input) (at 34.29 158.75 180) (fields_autoplaced)
-    (effects (font (size 1.27 1.27)) (justify right))
-  )
   (hierarchical_label "5V_HP" (shape input) (at 224.79 104.14 90) (fields_autoplaced)
     (effects (font (size 1.27 1.27)) (justify left))
   )
-  (hierarchical_label "5V_CLEAN" (shape input) (at 34.29 154.305 180) (fields_autoplaced)
-    (effects (font (size 1.27 1.27)) (justify right))
-  )
   (hierarchical_label "3V3_HP" (shape input) (at 224.155 36.195 90) (fields_autoplaced)
     (effects (font (size 1.27 1.27)) (justify left))
   )
-  (hierarchical_label "3V3_HP" (shape input) (at 34.29 145.415 180) (fields_autoplaced)
-    (effects (font (size 1.27 1.27)) (justify right))
-  )
   (symbol (lib_id "Device:C") (at 126.365 62.865 0) (mirror y) (unit 1)
     (in_bom yes) (on_board yes) (dnp no)
@@
     )
   )
-  (symbol (lib_id "Connector:TestPoint_Small") (at 37.465 145.415 0) (unit 1)
-    (in_bom yes) (on_board yes) (dnp no)
-    (property "Reference" "TP1" (at 39.37 144.78 0)
-      (effects (font (size 1.27 1.27)) (justify left) hide)
-    )
-    (property "Value" "3V3HP" (at 38.735 145.415 0)
-      (effects (font (size 1.27 1.27)) (justify left))
-    )
-    (property "Footprint" "!footprints:TestPoint_Pad_D1.0mm" (at 42.545 145.415 0)
-      (effects (font (size 1.27 1.27)) hide)
-    )
-    (property "Datasheet" "~" (at 42.545 145.415 0)
-      (effects (font (size 1.27 1.27)) hide)
-    )
-    (property "DPN" "" (at 37.465 145.415 0)
-      (effects (font (size 1.27 1.27)) hide)
-    )
-    (pin "1")
-    (instances
-      (project "backplane-concept"
-        (path "/1eedfbfd-a1b6-445d-9b0a-8fd3d481d4f1"
-          (reference "TP1") (unit 1)
-        )
-        (path "/1eedfbfd-a1b6-445d-9b0a-8fd3d481d4f1/87818b5d-e545-48ed-9242-b2d51bd0198b"
-          (reference "TP9") (unit 1)
-        )
-      )
-    )
-  )
   (symbol (lib_id "power:GND") (at 116.205 114.3 0) (unit 1)
     (in_bom yes) (on_board yes) (dnp no) (fields_autoplaced)
@@
         (path "/1eedfbfd-a1b6-445d-9b0a-8fd3d481d4f1/87818b5d-e545-48ed-9242-b2d51bd0198b"
           (reference "C8") (unit 1)
-        )
-      )
-    )
-  )
-  (symbol (lib_id "Connector:TestPoint_Small") (at 37.465 149.86 0) (unit 1)
-    (in_bom yes) (on_board yes) (dnp no)
-    (property "Reference" "TP1" (at 39.37 149.225 0)
-      (effects (font (size 1.27 1.27)) (justify left) hide)
-    )
-    (property "Value" "3V3C" (at 38.735 149.86 0)
-      (effects (font (size 1.27 1.27)) (justify left))
-    )
-    (property "Footprint" "!footprints:TestPoint_Pad_D1.0mm" (at 42.545 149.86 0)
-      (effects (font (size 1.27 1.27)) hide)
-    )
-    (property "Datasheet" "~" (at 42.545 149.86 0)
-      (effects (font (size 1.27 1.27)) hide)
-    )
-    (property "DPN" "" (at 37.465 149.86 0)
-      (effects (font (size 1.27 1.27)) hide)
-    )
-    (pin "1")
-    (instances
-      (project "backplane-concept"
-        (path "/1eedfbfd-a1b6-445d-9b0a-8fd3d481d4f1"
-          (reference "TP1") (unit 1)
-        )
-        (path "/1eedfbfd-a1b6-445d-9b0a-8fd3d481d4f1/87818b5d-e545-48ed-9242-b2d51bd0198b"
-          (reference "TP8") (unit 1)
-        )
-      )
-    )
-  )
-  (symbol (lib_id "Connector:TestPoint_Small") (at 37.465 140.97 0) (unit 1)
-    (in_bom yes) (on_board yes) (dnp no)
-    (property "Reference" "TP1" (at 39.37 140.335 0)
-      (effects (font (size 1.27 1.27)) (justify left) hide)
-    )
-    (property "Value" "VIN" (at 38.735 140.97 0)
-      (effects (font (size 1.27 1.27)) (justify left))
-    )
-    (property "Footprint" "!footprints:TestPoint_Pad_D1.0mm" (at 42.545 140.97 0)
-      (effects (font (size 1.27 1.27)) hide)
-    )
-    (property "Datasheet" "~" (at 42.545 140.97 0)
-      (effects (font (size 1.27 1.27)) hide)
-    )
-    (property "DPN" "" (at 37.465 140.97 0)
-      (effects (font (size 1.27 1.27)) hide)
-    )
-    (pin "1")
-    (instances
-      (project "backplane-concept"
-        (path "/1eedfbfd-a1b6-445d-9b0a-8fd3d481d4f1"
-          (reference "TP1") (unit 1)
-        )
-        (path "/1eedfbfd-a1b6-445d-9b0a-8fd3d481d4f1/87818b5d-e545-48ed-9242-b2d51bd0198b"
-          (reference "TP11") (unit 1)
         )
       )
@@
     )
   )
-  (symbol (lib_id "Connector:TestPoint_Small") (at 37.465 154.305 0) (unit 1)
-    (in_bom yes) (on_board yes) (dnp no)
-    (property "Reference" "TP1" (at 39.37 153.67 0)
-      (effects (font (size 1.27 1.27)) (justify left) hide)
-    )
-    (property "Value" "5VC" (at 38.735 154.305 0)
-      (effects (font (size 1.27 1.27)) (justify left))
-    )
-    (property "Footprint" "!footprints:TestPoint_Pad_D1.0mm" (at 42.545 154.305 0)
-      (effects (font (size 1.27 1.27)) hide)
-    )
-    (property "Datasheet" "~" (at 42.545 154.305 0)
-      (effects (font (size 1.27 1.27)) hide)
-    )
-    (property "DPN" "" (at 37.465 154.305 0)
-      (effects (font (size 1.27 1.27)) hide)
-    )
-    (pin "1")
-    (instances
-      (project "backplane-concept"
-        (path "/1eedfbfd-a1b6-445d-9b0a-8fd3d481d4f1"
-          (reference "TP1") (unit 1)
-        )
-        (path "/1eedfbfd-a1b6-445d-9b0a-8fd3d481d4f1/87818b5d-e545-48ed-9242-b2d51bd0198b"
-          (reference "TP7") (unit 1)
-        )
-      )
-    )
-  )
   (symbol (lib_id "Device:C") (at 127.635 109.22 0) (mirror y) (unit 1)
     (in_bom yes) (on_board yes) (dnp no)
@@
         )
       )
-    )
-  )
-  (symbol (lib_id "Connector:TestPoint_Small") (at 37.465 158.75 0) (unit 1)
-    (in_bom yes) (on_board yes) (dnp no)
-    (property "Reference" "TP1" (at 39.37 158.115 0)
-      (effects (font (size 1.27 1.27)) (justify left) hide)
-    )
-    (property "Value" "5VHP" (at 38.735 158.75 0)
-      (effects (font (size 1.27 1.27)) (justify left))
-    )
-    (property "Footprint" "!footprints:TestPoint_Pad_D1.0mm" (at 42.545 158.75 0)
-      (effects (font (size 1.27 1.27)) hide)
-    )
-    (property "Datasheet" "~" (at 42.545 158.75 0)
-      (effects (font (size 1.27 1.27)) hide)
-    )
-    (property "DPN" "" (at 37.465 158.75 0)
-      (effects (font (size 1.27 1.27)) hide)
-    )
-    (pin "1")
-    (instances
-      (project "backplane-concept"
-        (path "/1eedfbfd-a1b6-445d-9b0a-8fd3d481d4f1"
-          (reference "TP1") (unit 1)
-        )
-        (path "/1eedfbfd-a1b6-445d-9b0a-8fd3d481d4f1/87818b5d-e545-48ed-9242-b2d51bd0198b"
-          (reference "TP10") (unit 1)
-        )
-      )
